Commit message: Repair paths.

File: arm_description/hand.xacro (robot description, xacro)
@@ -12,5 +12,6 @@
       <visual>
         <geometry>
-          <mesh filename="file:///home/franz/catkin_ws/src/robocol_new_arm/meshes/visual/garra.stl" scale="0.01 0.01 0.01"/>
+          <mesh filename="file://$(arg robocol_new_arm)/meshes/visual/garra.stl" scale="0.01 0.01 0.01"/>
+          <!-- <mesh filename="file:///home/franz/catkin_ws/src/robocol_new_arm/meshes/visual/garra.stl" scale="0.01 0.01 0.01"/> -->
           <!-- <mesh filename="package://franka_description/meshes/visual/hand.dae"/> -->
         </geometry>

File: arm_description/robocol_arm.xacro (robot description, xacro)
@@ -12,5 +12,6 @@
       <visual>
         <geometry>
-          <mesh filename="file:///home/franz/catkin_ws/src/robocol_new_arm/meshes/visual/link0.stl" scale="0.01 0.01 0.01"/>
+          <mesh filename="file://$(arg robocol_new_arm)/meshes/visual/link0.dae" scale="0.01 0.01 0.01"/>
+          <!-- <mesh filename="file:///home/franz/catkin_ws/src/robocol_new_arm/meshes/visual/link0.stl" scale="0.01 0.01 0.01"/> -->
           <!-- <mesh filename="package://${description_pkg}/meshes/visual/link0.dae"/> -->
         </geometry>
@@ -25,5 +26,5 @@
       <visual>
         <geometry>
-          <mesh filename="file:///home/franz/catkin_ws/src/robocol_new_arm/meshes/visual/link1.stl" scale="0.01 0.01 0.01"/>
+          <mesh filename="file://$(arg robocol_new_arm)/meshes/visual/link1.dae" scale="0.01 0.01 0.01"/>
           <!-- <mesh filename="package://${description_pkg}/meshes/visual/link1.dae"/> -->
         </geometry>
@@ -46,5 +47,5 @@
       <visual>
         <geometry>
-          <mesh filename="file:///home/franz/catkin_ws/src/robocol_new_arm/meshes/visual/link2.stl" scale="0.01 0.01 0.01"/>
+          <mesh filename="file://$(arg robocol_new_arm)/meshes/visual/link2.dae" scale="0.01 0.01 0.01"/>
           <!-- <mesh filename="package://${description_pkg}/meshes/visual/link2.dae"/> -->
         </geometry>
@@ -67,5 +68,5 @@
       <visual>
         <geometry>
-          <mesh filename="file:///home/franz/catkin_ws/src/robocol_new_arm/meshes/visual/link3.stl" scale="0.01 0.01 0.01"/>
+          <mesh filename="file://$(arg robocol_new_arm)/meshes/visual/link3.dae" scale="0.01 0.01 0.01"/>
           <!-- <mesh filename="package://${description_pkg}/meshes/visual/link3.dae"/> -->
         </geometry>
@@ -88,5 +89,5 @@
       <visual>
         <geometry>
-          <mesh filename="file:///home/franz/catkin_ws/src/robocol_new_arm/meshes/visual/link4.stl" scale="0.01 0.01 0.01"/>
+          <mesh filename="file://$(arg robocol_new_arm)/meshes/visual/link4.dae" scale="0.01 0.01 0.01"/>
           <!-- <mesh filename="package://${description_pkg}/meshes/visual/link4.dae"/> -->
         </geometry>
@@ -109,6 +110,6 @@
       <visual>
         <geometry>
-          <mesh filename="file:///home/franz/catkin_ws/src/robocol_new_arm/meshes/visual/link5.stl" scale="0.01 0.01 0.01"/>
-          <mesh filename="package://${description_pkg}/meshes/visual/link5.dae"/>
+          <mesh filename="file://$(arg robocol_new_arm)/meshes/visual/link5.dae" scale="0.01 0.01 0.01"/>
+          <!-- <mesh filename="package://${description_pkg}/meshes/visual/link5.dae"/>  -->
         </geometry>
       </visual>
