Commit message: Push to start Documentation.

File: arm_description/robocol_arm.xacro (robot description, xacro)
@@ -63,5 +63,5 @@
       <child link="${arm_id}_link2"/>
       <axis xyz="0 0 1"/>
-      <limit effort="87" lower="-1.7628" upper="1.7628" velocity="2.1750"/>
+      <limit effort="87" lower="-2.7628" upper="2.7628" velocity="2.1750"/>
     </joint>
     <link name="${arm_id}_link3">

File: urdf/robocol_arm.urdf (robot description, URDF)
Before this commit: robot robocol, 7 links, 6 joints
Joints:
- joint robocol_joint2: limit lower=-1.75 upper=1.75 effort=87 velocity=2.3925 -> lower=-2.75 upper=2.75 effort=87 velocity=2.3925
- joint robocol_joint3: limit lower=-1.87 upper=2.76 effort=87 velocity=2.3925 -> lower=-2.87 upper=2.76 effort=87 velocity=2.3925
