Commit message: Hand changes.

File: arm_description/hand_WORKING.xacro (robot description, xacro)
@@ -9,30 +9,30 @@
       </joint>
     </xacro:unless>
-    <material name="hand_mat">
-      <color rgba="0.9 0.6 0 1"/>
-    </material>
     <link name="${ns}_hand">
       <visual>
         <geometry>
-          <mesh filename="package://robocol_new_arm/meshes/visual/hand.stl" scale="0.1 0.1 0.1"/>
+          <mesh filename="file://$(arg robocol_new_arm)/meshes/visual/garra.stl" scale="0.01 0.01 0.01"/>
+          <!-- <mesh filename="file:///home/franz/catkin_ws/src/robocol_new_arm/meshes/visual/garra.stl" scale="0.01 0.01 0.01"/> -->
+          <!-- <mesh filename="package://franka_description/meshes/visual/hand.dae"/> -->
         </geometry>
-        <material name="joints_mat"/>
+      </visual>
+      <!--
+      <collision>
+        <geometry>
+          <mesh filename="package://franka_description/meshes/collision/hand.stl"/>
+        </geometry>
+      </collision>
+       -->
+    </link>
+    <!--
+    <link name="${ns}_leftfinger">
+      <visual>
+        <geometry>
+          <mesh filename="package://franka_description/meshes/visual/finger.dae"/>
+        </geometry>
       </visual>
       <collision>
         <geometry>
-          <mesh filename="package://robocol_new_arm/meshes/collision/hand.stl" scale="0.1 0.1 0.1"/>
-        </geometry>
-      </collision>
-    </link>
-    <link name="${ns}_leftfinger">
-      <visual>
-        <geometry>
-          <mesh filename="package://robocol_new_arm/meshes/visual/finger.stl" scale="0.1 0.1 0.1"/>
-        </geometry>
-        <material name="joints_mat"/>
-      </visual>
-      <collision>
-        <geometry>
-          <mesh filename="package://robocol_new_arm/meshes/collision/finger.stl" scale="0.1 0.1 0.1"/>
+          <mesh filename="package://franka_description/meshes/collision/finger.stl"/>
         </geometry>
       </collision>
@@ -42,12 +42,11 @@
         <origin xyz="0 0 0" rpy="0 0 ${pi}"/>
         <geometry>
-          <mesh filename="package://robocol_new_arm/meshes/visual/finger.stl" scale="0.1 0.1 0.1"/>
+          <mesh filename="package://franka_description/meshes/visual/finger.dae"/>
         </geometry>
-        <material name="joints_mat"/>
       </visual>
       <collision>
         <origin xyz="0 0 0" rpy="0 0 ${pi}"/>
         <geometry>
-          <mesh filename="package://robocol_new_arm/meshes/collision/finger.stl" scale="0.1 0.1 0.1"/>
+          <mesh filename="package://franka_description/meshes/collision/finger.stl"/>
         </geometry>
       </collision>
@@ -56,16 +55,17 @@
       <parent link="${ns}_hand"/>
       <child link="${ns}_leftfinger"/>
-      <origin xyz="-0.5 0 0.65" rpy="0 ${pi/2} 0"/>
-      <axis xyz="0 0 1"/>
-      <limit effort="20" lower="0.0" upper="0.28" velocity="0.2"/>
+      <origin xyz="0 0 0.0584" rpy="0 0 0"/>
+      <axis xyz="0 1 0"/>
+      <limit effort="20" lower="0.0" upper="0.04" velocity="0.2"/>
     </joint>
     <joint name="${ns}_finger_joint2" type="prismatic">
       <parent link="${ns}_hand"/>
       <child link="${ns}_rightfinger"/>
-      <origin xyz="0.5 0 0.65" rpy="0 ${-pi/2} 0"/>
-      <axis xyz="0 0 1"/>
-      <limit effort="20" lower="0.0" upper="0.28" velocity="0.2"/>
+      <origin xyz="0 0 0.0584" rpy="0 0 0"/>
+      <axis xyz="0 -1 0"/>
+      <limit effort="20" lower="0.0" upper="0.04" velocity="0.2"/>
       <mimic joint="${ns}_finger_joint1" />
     </joint>
+    -->
   </xacro:macro>
 </robot>

File: arm_description/robocol_arm.xacro (robot description, xacro)
@@ -9,173 +9,134 @@
       </joint>
     </xacro:unless>
+    <material name="joints_mat">
+      <color rgba="0.75 0.6 0.3 1"/>
+    </material>
     <link name="${arm_id}_link0">
       <visual>
         <geometry>
-          <mesh filename="file://$(arg robocol_new_arm)/meshes/visual/link0.dae" scale="0.01 0.01 0.01"/>
-          <!-- <mesh filename="file:///home/franz/catkin_ws/src/robocol_new_arm/meshes/visual/link0.stl" scale="0.01 0.01 0.01"/> -->
-          <!-- <mesh filename="package://${description_pkg}/meshes/visual/link0.dae"/> -->
+          <mesh filename="package://${description_pkg}/meshes/visual/link0.stl" scale="0.1 0.1 0.1"/>
         </geometry>
+        <material name="joints_mat"/>
       </visual>
-      <!-- <collision>
+      <collision>
         <geometry>
-          <mesh filename="package://${description_pkg}/meshes/collision/link0.stl"/>
+          <mesh filename="package://${description_pkg}/meshes/collision/link0.stl" scale="0.1 0.1 0.1"/>
         </geometry>
-      </collision> -->
+      </collision>
     </link>
     <link name="${arm_id}_link1">
       <visual>
         <geometry>
-          <mesh filename="file://$(arg robocol_new_arm)/meshes/visual/link1.dae" scale="0.01 0.01 0.01"/>
-          <!-- <mesh filename="package://${description_pkg}/meshes/visual/link1.dae"/> -->
+          <mesh filename="package://${description_pkg}/meshes/visual/link1.stl" scale="0.1 0.1 0.1"/>
         </geometry>
+        <material name="joints_mat"/>
       </visual>
-      <!-- <collision>
+      <collision>
         <geometry>
-          <mesh filename="package://${description_pkg}/meshes/collision/link1.stl"/>
+          <mesh filename="package://${description_pkg}/meshes/collision/link1.stl" scale="0.1 0.1 0.1"/>
         </geometry>
-      </collision> -->
+      </collision>
     </link>
     <joint name="${arm_id}_joint1" type="revolute">
-      <!-- <safety_controller k_position="100.0" k_velocity="40.0" soft_lower_limit="-2.8973" soft_upper_limit="2.8973"/> -->
-      <origin rpy="0 0 0" xyz="0 0 0.333"/>
+      <safety_controller k_position="100.0" k_velocity="40.0" soft_lower_limit="-3" soft_upper_limit="3"/>
+      <origin rpy="0 0 0" xyz="0 0 1.4"/>
       <parent link="${arm_id}_link0"/>
       <child link="${arm_id}_link1"/>
       <axis xyz="0 0 1"/>
-      <limit effort="87" lower="-2.8973" upper="2.8973" velocity="2.1750"/>
+      <limit effort="87" lower="-3" upper="3" velocity="2.1750"/>
     </joint>
     <link name="${arm_id}_link2">
       <visual>
         <geometry>
-          <mesh filename="file://$(arg robocol_new_arm)/meshes/visual/link2.dae" scale="0.01 0.01 0.01"/>
-          <!-- <mesh filename="package://${description_pkg}/meshes/visual/link2.dae"/> -->
+          <mesh filename="package://${description_pkg}/meshes/visual/link2.stl" scale="0.1 0.1 0.1"/>
         </geometry>
+        <material name="joints_mat"/>
       </visual>
-      <!-- <collision>
+      <collision>
         <geometry>
-          <mesh filename="package://${description_pkg}/meshes/collision/link2.stl"/>
+          <mesh filename="package://${description_pkg}/meshes/collision/link2.stl" scale="0.1 0.1 0.1"/>
         </geometry>
-      </collision> -->
+      </collision>
     </link>
     <joint name="${arm_id}_joint2" type="revolute">
-      <!-- <safety_controller k_position="100.0" k_velocity="40.0" soft_lower_limit="-1.7628" soft_upper_limit="1.7628"/> -->
-      <origin rpy="${-pi/2} 0 0" xyz="0 0 0"/>
+      <safety_controller k_position="100.0" k_velocity="40.0" soft_lower_limit="-1.7628" soft_upper_limit="2.5"/>
+      <origin rpy="0 ${-pi/2} 0" xyz="0.74 -0.55 1.2"/>
       <parent link="${arm_id}_link1"/>
       <child link="${arm_id}_link2"/>
-      <axis xyz="0 0 1"/>
-      <limit effort="87" lower="-2.7628" upper="2.7628" velocity="2.1750"/>
+      <axis xyz="0 1 0"/>
+      <limit effort="87" lower="-1.7628" upper="2.5" velocity="2.1750"/>
     </joint>
     <link name="${arm_id}_link3">
       <visual>
         <geometry>
-          <mesh filename="file://$(arg robocol_new_arm)/meshes/visual/link3.dae" scale="0.01 0.01 0.01"/>
-          <!-- <mesh filename="package://${description_pkg}/meshes/visual/link3.dae"/> -->
+          <mesh filename="package://${description_pkg}/meshes/visual/link3.stl" scale="0.1 0.1 0.1"/>
         </geometry>
+        <material name="joints_mat"/>
       </visual>
-      <!-- <collision>
+      <collision>
         <geometry>
-          <mesh filename="package://${description_pkg}/meshes/collision/link3.stl"/>
+          <mesh filename="package://${description_pkg}/meshes/collision/link3.stl" scale="0.1 0.1 0.1"/>
         </geometry>
-      </collision> -->
+      </collision>
     </link>
     <joint name="${arm_id}_joint3" type="revolute">
-      <!-- <safety_controller k_position="100.0" k_velocity="40.0" soft_lower_limit="-2.8973" soft_upper_limit="2.8973"/> -->
-      <origin rpy="${pi/2} 0 0" xyz="0 -0.316 0"/>
+      <safety_controller k_position="100.0" k_velocity="40.0" soft_lower_limit="-2.6" soft_upper_limit="2.6"/>
+      <origin rpy="0 ${pi/2} 0" xyz="2.5 0 0"/>
       <parent link="${arm_id}_link2"/>
       <child link="${arm_id}_link3"/>
-      <axis xyz="0 0 1"/>
-      <limit effort="87" lower="-2.8973" upper="2.8973" velocity="2.1750"/>
+      <axis xyz="0 1 0"/>
+      <limit effort="87" lower="-2.6" upper="2.6" velocity="2.1750"/>
     </joint>
     <link name="${arm_id}_link4">
       <visual>
         <geometry>
-          <mesh filename="file://$(arg robocol_new_arm)/meshes/visual/link4.dae" scale="0.01 0.01 0.01"/>
-          <!-- <mesh filename="package://${description_pkg}/meshes/visual/link4.dae"/> -->
+          <mesh filename="package://${description_pkg}/meshes/visual/link4.stl" scale="0.1 0.1 0.1"/>
         </geometry>
+        <material name="joints_mat"/>
       </visual>
-      <!-- <collision>
+      <collision>
         <geometry>
-          <mesh filename="package://${description_pkg}/meshes/collision/link4.stl"/>
+          <mesh filename="package://${description_pkg}/meshes/collision/link4.stl" scale="0.1 0.1 0.1"/>
         </geometry>
-      </collision> -->
+      </collision>
     </link>
     <joint name="${arm_id}_joint4" type="revolute">
-      <!-- <safety_controller k_position="100.0" k_velocity="40.0" soft_lower_limit="-3.0718" soft_upper_limit="-0.0698"/> -->
-      <origin rpy="${pi/2} 0 0" xyz="0.0825 0 0"/>
+      <safety_controller k_position="100.0" k_velocity="40.0" soft_lower_limit="-2.5" soft_upper_limit="2.5"/>
+      <origin rpy="0 0 ${-pi/2}" xyz="-0.05 0.55 1.5"/>
       <parent link="${arm_id}_link3"/>
       <child link="${arm_id}_link4"/>
       <axis xyz="0 0 1"/>
-      <limit effort="87" lower="-3.0718" upper="-0.0698" velocity="2.1750"/>
+      <limit effort="87" lower="-2.5" upper="2.5" velocity="2.1750"/>
     </joint>
     <link name="${arm_id}_link5">
       <visual>
         <geometry>
-          <mesh filename="file://$(arg robocol_new_arm)/meshes/visual/link5.dae" scale="0.01 0.01 0.01"/>
-          <!-- <mesh filename="package://${description_pkg}/meshes/visual/link5.dae"/>  -->
+          <mesh filename="package://${description_pkg}/meshes/visual/link5.stl" scale="0.1 0.1 0.1"/>
         </geometry>
-      </visual>
-      <!-- <collision>
-        <geometry>
-          <mesh filename="package://${description_pkg}/meshes/collision/link5.stl"/>
-        </geometry>
-      </collision> -->
-    </link>
-    <joint name="${arm_id}_joint5" type="revolute">
-      <!-- <safety_controller k_position="100.0" k_velocity="40.0" soft_lower_limit="-2.8973" soft_upper_limit="2.8973"/> -->
-      <origin rpy="${-pi/2} 0 0" xyz="-0.0825 0.384 0"/>
-      <parent link="${arm_id}_link4"/>
-      <child link="${arm_id}_link5"/>
-      <axis xyz="0 0 1"/>
-      <limit effort="12" lower="-2.8973" upper="2.8973" velocity="2.6100"/>
-    </joint>
-    <link name="${arm_id}_link6"/>
-    <!-- <link name="${arm_id}_link6">
-      <visual>
-        <geometry>
-          <mesh filename="file:///home/franz/catkin_ws/src/robocol_new_arm/meshes/visual/link6.stl" scale="0.1 0.1 0.1"/>
-          <mesh filename="package://${description_pkg}/meshes/visual/link6.dae"/>
-        </geometry>
+        <material name="joints_mat"/>
       </visual>
       <collision>
         <geometry>
-          <mesh filename="package://${description_pkg}/meshes/collision/link6.stl"/>
+          <mesh filename="package://${description_pkg}/meshes/collision/link5.stl" scale="0.1 0.1 0.1"/>
         </geometry>
       </collision>
     </link>
+    <joint name="${arm_id}_joint5" type="revolute">
+      <safety_controller k_position="100.0" k_velocity="40.0" soft_lower_limit="-2.5" soft_upper_limit="2.5"/>
+      <origin rpy="0 0 0" xyz="0.42 0.04 1.53"/>
+      <parent link="${arm_id}_link4"/>
+      <child link="${arm_id}_link5"/>
+      <axis xyz="1 0 0"/>
+      <limit effort="12" lower="-2.5" upper="2.5" velocity="2.6100"/>
+    </joint>
+    <link name="${arm_id}_link6"/>
     <joint name="${arm_id}_joint6" type="revolute">
-      <safety_controller k_position="100.0" k_velocity="40.0" soft_lower_limit="-0.0175" soft_upper_limit="3.7525"/>
-      <origin rpy="${pi/2} 0 0" xyz="0 0 0"/>
+      <safety_controller k_position="100.0" k_velocity="40.0" soft_lower_limit="-3" soft_upper_limit="3"/>
+      <origin rpy="0 0 -0.8" xyz="-0.3 0.1 1.4"/>
       <parent link="${arm_id}_link5"/>
       <child link="${arm_id}_link6"/>
       <axis xyz="0 0 1"/>
-      <limit effort="12" lower="-0.0175" upper="3.7525" velocity="2.6100"/>
+      <limit effort="12" lower="-3" upper="3" velocity="2.6100"/>
     </joint>
-    <link name="${arm_id}_link7">
-      <visual>
-        <geometry>
-          <mesh filename="file:///home/franz/catkin_ws/src/robocol_new_arm/meshes/visual/link7.stl" scale="0.1 0.1 0.1"/>
-          <mesh filename="package://${description_pkg}/meshes/visual/link7.dae"/>
-        </geometry>
-      </visual>
-      <collision>
-        <geometry>
-          <mesh filename="package://${description_pkg}/meshes/collision/link7.stl"/>
-        </geometry>
-      </collision>
-    </link>
-    <joint name="${arm_id}_joint7" type="revolute">
-      <safety_controller k_position="100.0" k_velocity="40.0" soft_lower_limit="-2.8973" soft_upper_limit="2.8973"/>
-      <origin rpy="${pi/2} 0 0" xyz="0.088 0 0"/>
-      <parent link="${arm_id}_link6"/>
-      <child link="${arm_id}_link7"/>
-      <axis xyz="0 0 1"/>
-      <limit effort="12" lower="-2.8973" upper="2.8973" velocity="2.6100"/>
-    </joint>
-    <link name="${arm_id}_link8"/>
-    <joint name="${arm_id}_joint8" type="fixed">
-      <origin rpy="0 0 0" xyz="0 0 0.107"/>
-      <parent link="${arm_id}_link7"/>
-      <child link="${arm_id}_link8"/>
-      <axis xyz="0 0 0"/>
-    </joint> -->
   </xacro:macro>
 </robot>

File: arm_description/robocol_arm_hand.urdf.xacro (robot description, xacro)
@@ -4,4 +4,4 @@
   <xacro:include filename="$(find robocol_new_arm)/arm_description/hand.xacro"/>
   <xacro:robocol_arm />
-  <xacro:hand ns="robocol" rpy="0 0 ${-pi/4}" connected_to="robocol_link5"/>
+  <xacro:hand ns="robocol" rpy="0 0 ${-pi/4}" connected_to="robocol_link6"/>
 </robot>

File: config/hand_LAST.xacro (robot description, xacro)
@@ -9,15 +9,15 @@
     <group name="hand">
       <link name="robocol_hand" />
-      <link name="robocol_leftfinger" />
-      <link name="robocol_rightfinger" />
-      <joint name="robocol_finger_joint1" />
-      <passive_joint name="robocol_finger_joint2" />
+      <!-- <link name="robocol_leftfinger" /> -->
+      <!-- <link name="robocol_rightfinger" /> -->
+      <!-- <joint name="robocol_finger_joint1" /> -->
+      <!-- <passive_joint name="robocol_finger_joint2" /> -->
     </group>
     <!--GROUP STATES: Purpose: Define a named state for a particular group, in terms of joint values. This is useful to define states like 'folded arms'-->
     <!--END EFFECTOR: Purpose: Represent information about an end effector.-->
     <!--DISABLE COLLISIONS: By default it is assumed that any link of the robot could potentially come into collision with any other link in the robot. This tag disables collision checking between a specified pair of links. -->
-    <disable_collisions link1="robocol_hand" link2="robocol_leftfinger" reason="Adjacent" />
-    <disable_collisions link1="robocol_hand" link2="robocol_rightfinger" reason="Adjacent" />
-    <disable_collisions link1="robocol_leftfinger" link2="robocol_rightfinger" reason="Default" />
+    <!-- <disable_collisions link1="robocol_hand" link2="robocol_leftfinger" reason="Adjacent" /> -->
+    <!-- <disable_collisions link1="robocol_hand" link2="robocol_rightfinger" reason="Adjacent" /> -->
+    <!-- <disable_collisions link1="robocol_leftfinger" link2="robocol_rightfinger" reason="Default" /> -->
   </xacro:macro>
 </robot>

File: config/robocol_arm.xacro (robot description, xacro)
@@ -8,5 +8,5 @@
     <!--SUBGROUPS: Groups can also be formed by referencing to already defined group names-->
     <group name="robocol_arm">
-      <chain base_link="robocol_link0" tip_link="robocol_hand" />
+      <chain base_link="robocol_link0" tip_link="robocol_link6" />
     </group>
     <!--GROUP STATES: Purpose: Define a named state for a particular group, in terms of joint values. This is useful to define states like 'folded arms'-->
@@ -17,5 +17,5 @@
       <joint name="robocol_joint4" value="0" />
       <joint name="robocol_joint5" value="1.19" />
-      <joint name="robocol_joint6" value="0" />
+      <!-- <joint name="robocol_joint6" value="0" /> -->
     </group_state>
     <group_state name="ready" group="robocol_arm">
@@ -25,5 +25,5 @@
       <joint name="robocol_joint4" value="0" />
       <joint name="robocol_joint5" value="-0.78" />
-      <joint name="robocol_joint6" value="1.57" />
+      <!-- <joint name="robocol_joint6" value="1.57" /> -->
     </group_state>
     <group_state name="pick" group="robocol_arm">
@@ -33,5 +33,5 @@
       <joint name="robocol_joint4" value="0" />
       <joint name="robocol_joint5" value="0" />
-      <joint name="robocol_joint6" value="1.57" />
+      <!-- <joint name="robocol_joint6" value="1.57" /> -->
     </group_state>
     <group_state name="place_right" group="robocol_arm">
@@ -41,5 +41,5 @@
       <joint name="robocol_joint4" value="0" />
       <joint name="robocol_joint5" value="-0.95" />
-      <joint name="robocol_joint6" value="2.95" />
+      <!-- <joint name="robocol_joint6" value="2.95" /> -->
     </group_state>
     <group_state name="place_left" group="robocol_arm">
@@ -49,5 +49,5 @@
       <joint name="robocol_joint4" value="0" />
       <joint name="robocol_joint5" value="-0.95" />
-      <joint name="robocol_joint6" value="2.95" />
+      <!-- <joint name="robocol_joint6" value="2.95" /> -->
     </group_state>
     <group_state name="all_0" group="robocol_arm">
@@ -57,9 +57,9 @@
       <joint name="robocol_joint4" value="0" />
       <joint name="robocol_joint5" value="0" />
-      <joint name="robocol_joint6" value="0" />
+      <!-- <joint name="robocol_joint6" value="0" /> -->
     </group_state>
     <!--END EFFECTOR: Purpose: Represent information about an end effector.-->
     <!--VIRTUAL JOINT: Purpose: this element defines a virtual joint between a robot link and an external frame of reference (considered fixed with respect to the robot)-->
-    <!-- <virtual_joint name="virtual_joint" type="floating" parent_frame="world" child_link="robocol_link0" /> -->
+    <virtual_joint name="virtual_joint" type="floating" parent_frame="world" child_link="robocol_link0" />
     <!--DISABLE COLLISIONS: By default it is assumed that any link of the robot could potentially come into collision with any other link in the robot. This tag disables collision checking between a specified pair of links. -->
     <disable_collisions link1="robocol_link0" link2="robocol_link1" reason="Adjacent" />
@@ -80,10 +80,7 @@
     <!-- <disable_collisions link1="robocol_link3" link2="robocol_link5" reason="Never" /> -->
     <!-- <disable_collisions link1="robocol_link3" link2="robocol_link6" reason="Never" /> -->
-    <!-- <disable_collisions link1="robocol_link3" link2="robocol_link7" reason="Never" /> -->
     <!-- <disable_collisions link1="robocol_link4" link2="robocol_link5" reason="Adjacent" /> -->
     <!-- <disable_collisions link1="robocol_link4" link2="robocol_link6" reason="Never" /> -->
-    <!-- <disable_collisions link1="robocol_link4" link2="robocol_link7" reason="Never" /> -->
     <!-- <disable_collisions link1="robocol_link5" link2="robocol_link6" reason="Adjacent" /> -->
-    <!-- <disable_collisions link1="robocol_link6" link2="pandrobocola_link7" reason="Adjacent" /> -->
   </xacro:macro>
 </robot>
