Commit message: Hand changes.

File: config/robocol_arm_hand.srdf.xacro (robot description, xacro)
@@ -18,30 +18,26 @@
     <group name="robocol_arm" />
     <group name="hand" />
-    <!-- <group name="partial_robocol_arm" /> -->
   </group>
-  <!--GROUP STATES: Purpose: Define a named state for a particular group, in terms of joint values. This is useful to define states like 'folded arms'-->
-  <group_state name="ready" group="robocol_arm_hand">
-    <joint name="robocol_joint1" value="0" />
-    <joint name="robocol_joint2" value="-1.75" />
-    <joint name="robocol_joint3" value="2.62" />
-    <joint name="robocol_joint4" value="0" />
-    <joint name="robocol_joint5" value="1.19" />
-    <joint name="robocol_joint6" value="0" />
+  <group_state name="open" group="hand">
+    <joint name="robocol_finger_joint1" value="0.035" />
+    <joint name="robocol_finger_joint2" value="0.035" />
+  </group_state>
+  <group_state name="close" group="hand">
+    <joint name="robocol_finger_joint1" value="0" />
+    <joint name="robocol_finger_joint2" value="0" />
   </group_state>
   <!--END EFFECTOR: Purpose: Represent information about an end effector.-->
-  <end_effector name="hand" parent_link="robocol_link5" group="hand" parent_group="robocol_arm" />
+  <end_effector name="hand" parent_link="robocol_link6" group="hand" parent_group="robocol_arm" />
   <!--DISABLE COLLISIONS: By default it is assumed that any link of the robot could potentially come into collision with any other link in the robot. This tag disables collision checking between a specified pair of links. -->
   <disable_collisions link1="robocol_hand" link2="robocol_link3" reason="Never" />
   <disable_collisions link1="robocol_hand" link2="robocol_link4" reason="Never" />
-  <!-- <disable_collisions link1="robocol_hand" link2="robocol_link6" reason="Never" /> -->
+  <disable_collisions link1="robocol_hand" link2="robocol_link6" reason="Never" />
   <disable_collisions link1="robocol_hand" link2="robocol_link5" reason="Adjacent" />
-  <!-- <disable_collisions link1="robocol_hand" link2="robocol_link6" reason="Adjacent" /> -->
-  <!-- <disable_collisions link1="robocol_leftfinger" link2="robocol_link3" reason="Never" /> -->
-  <!-- <disable_collisions link1="robocol_leftfinger" link2="robocol_link4" reason="Never" /> -->
-  <!-- <disable_collisions link1="robocol_leftfinger" link2="robocol_link6" reason="Never" /> -->
-  <!-- <disable_collisions link1="robocol_leftfinger" link2="robocol_link7" reason="Never" /> -->
-  <!-- <disable_collisions link1="robocol_link3" link2="robocol_rightfinger" reason="Never" /> -->
-  <!-- <disable_collisions link1="robocol_link4" link2="robocol_rightfinger" reason="Never" /> -->
-  <!-- <disable_collisions link1="robocol_link6" link2="robocol_rightfinger" reason="Never" /> -->
-  <!-- <disable_collisions link1="robocol_link7" link2="robocol_rightfinger" reason="Never" /> -->
+  <disable_collisions link1="robocol_hand" link2="robocol_link6" reason="Adjacent" />
+  <disable_collisions link1="robocol_leftfinger" link2="robocol_link3" reason="Never" />
+  <disable_collisions link1="robocol_leftfinger" link2="robocol_link4" reason="Never" />
+  <disable_collisions link1="robocol_leftfinger" link2="robocol_link6" reason="Never" />
+  <disable_collisions link1="robocol_link3" link2="robocol_rightfinger" reason="Never" />
+  <disable_collisions link1="robocol_link4" link2="robocol_rightfinger" reason="Never" />
+  <disable_collisions link1="robocol_link6" link2="robocol_rightfinger" reason="Never" />
 </robot>
