Commit message: Changes in URDF.

File: urdf/robocol_arm.urdf (robot description, URDF)
Before this commit: robot robocol, 7 links, 6 joints
Links:
- link robocol_hand: geometry visual mesh filename=file://$(arg robocol_new_arm)/meshes/visual/hand.stl scale=0.1 0.1 0.1
- link robocol_link0: geometry visual mesh filename=file://$(arg robocol_new_arm)/meshes/visual/link0.stl scale=0.1 0.1 0.1
- link robocol_link1: geometry visual mesh filename=file://$(arg robocol_new_arm)/meshes/visual/link1.stl scale=0.1 0.1 0.1
- link robocol_link2: geometry visual mesh filename=file://$(arg robocol_new_arm)/meshes/visual/link2.stl scale=0.1 0.1 0.1
- link robocol_link3: geometry visual mesh filename=file://$(arg robocol_new_arm)/meshes/visual/link3.stl scale=0.1 0.1 0.1
- link robocol_link4: geometry visual mesh filename=file://$(arg robocol_new_arm)/meshes/visual/link4.stl scale=0.1 0.1 0.1
- link robocol_link5: geometry visual mesh filename=file://$(arg robocol_new_arm)/meshes/visual/link5.stl scale=0.1 0.1 0.1

Commit message: Path Changes in URDF.

File: urdf/robocol_arm.urdf (robot description, URDF)
Before this commit: robot robocol, 7 links, 6 joints
Links:
- link robocol_hand: geometry visual mesh filename=file://$(arg robocol_new_arm)meshes/visual/hand.stl scale=0.1 0.1 0.1
- link robocol_link0: geometry visual mesh filename=file://$(arg robocol_new_arm)meshes/visual/link0.stl scale=0.1 0.1 0.1
- link robocol_link1: geometry visual mesh filename=file://$(arg robocol_new_arm)meshes/visual/link1.stl scale=0.1 0.1 0.1
- link robocol_link2: geometry visual mesh filename=file://$(arg robocol_new_arm)meshes/visual/link2.stl scale=0.1 0.1 0.1
- link robocol_link3: geometry visual mesh filename=file://$(arg robocol_new_arm)meshes/visual/link3.stl scale=0.1 0.1 0.1
- link robocol_link4: geometry visual mesh filename=file://$(arg robocol_new_arm)meshes/visual/link4.stl scale=0.1 0.1 0.1
- link robocol_link5: geometry visual mesh filename=file://$(arg robocol_new_arm)meshes/visual/link5.stl scale=0.1 0.1 0.1

Commit message: Final Repair Paths

File: urdf/robocol_arm.urdf (robot description, URDF)
Before this commit: robot robocol, 7 links, 6 joints
Links:
- link robocol_hand: geometry visual mesh filename=package://robocol_new_arm/meshes/visual/hand.stl scale=0.1 0.1 0.1
- link robocol_link0: geometry visual mesh filename=package://robocol_new_arm/meshes/visual/link0.stl scale=0.1 0.1 0.1
- link robocol_link1: geometry visual mesh filename=package://robocol_new_arm/meshes/visual/link1.stl scale=0.1 0.1 0.1
- link robocol_link2: geometry visual mesh filename=package://robocol_new_arm/meshes/visual/link2.stl scale=0.1 0.1 0.1
- link robocol_link3: geometry visual mesh filename=package://robocol_new_arm/meshes/visual/link3.stl scale=0.1 0.1 0.1
- link robocol_link4: geometry visual mesh filename=package://robocol_new_arm/meshes/visual/link4.stl scale=0.1 0.1 0.1
- link robocol_link5: geometry visual mesh filename=package://robocol_new_arm/meshes/visual/link5.stl scale=0.1 0.1 0.1

Commit message: Last changes

File: urdf/robocol_arm.urdf (robot description, URDF)
Before this commit: robot robocol, 7 links, 6 joints
Joints:
- joint robocol_joint5: limit lower=-2.39 upper=1.75 effort=12 velocity=2.8710 -> lower=-2.39 upper=2.7 effort=12 velocity=2.8710
