Commit message: Major Changes
Major changes to robocol arm for it to work correctly.

File: config/robocol_arm.xacro (robot description, xacro)
@@ -11,5 +11,45 @@
     </group>
     <!--GROUP STATES: Purpose: Define a named state for a particular group, in terms of joint values. This is useful to define states like 'folded arms'-->
+    <group_state name="rest" group="robocol_arm">
+      <joint name="robocol_joint1" value="0" />
+      <joint name="robocol_joint2" value="-1.75" />
+      <joint name="robocol_joint3" value="2.62" />
+      <joint name="robocol_joint4" value="0" />
+      <joint name="robocol_joint5" value="1.19" />
+      <joint name="robocol_joint6" value="0" />
+    </group_state>
     <group_state name="ready" group="robocol_arm">
+      <joint name="robocol_joint1" value="0" />
+      <joint name="robocol_joint2" value="-0.78" />
+      <joint name="robocol_joint3" value="1.57" />
+      <joint name="robocol_joint4" value="0" />
+      <joint name="robocol_joint5" value="-0.78" />
+      <joint name="robocol_joint6" value="1.57" />
+    </group_state>
+    <group_state name="pick" group="robocol_arm">
+      <joint name="robocol_joint1" value="0" />
+      <joint name="robocol_joint2" value="1.7" />
+      <joint name="robocol_joint3" value="1.4" />
+      <joint name="robocol_joint4" value="0" />
+      <joint name="robocol_joint5" value="0" />
+      <joint name="robocol_joint6" value="1.57" />
+    </group_state>
+    <group_state name="place_right" group="robocol_arm">
+      <joint name="robocol_joint1" value="-1.57" />
+      <joint name="robocol_joint2" value="0" />
+      <joint name="robocol_joint3" value="2.17" />
+      <joint name="robocol_joint4" value="0" />
+      <joint name="robocol_joint5" value="-0.95" />
+      <joint name="robocol_joint6" value="2.95" />
+    </group_state>
+    <group_state name="place_left" group="robocol_arm">
+      <joint name="robocol_joint1" value="1.57" />
+      <joint name="robocol_joint2" value="0" />
+      <joint name="robocol_joint3" value="2.17" />
+      <joint name="robocol_joint4" value="0" />
+      <joint name="robocol_joint5" value="-0.95" />
+      <joint name="robocol_joint6" value="2.95" />
+    </group_state>
+    <group_state name="all_0" group="robocol_arm">
       <joint name="robocol_joint1" value="0" />
       <joint name="robocol_joint2" value="0" />

File: config/robocol_arm_hand.srdf.xacro (robot description, xacro)
@@ -23,8 +23,9 @@
   <group_state name="ready" group="robocol_arm_hand">
     <joint name="robocol_joint1" value="0" />
-    <joint name="robocol_joint2" value="0" />
-    <joint name="robocol_joint3" value="0" />
+    <joint name="robocol_joint2" value="-1.75" />
+    <joint name="robocol_joint3" value="2.62" />
     <joint name="robocol_joint4" value="0" />
-    <joint name="robocol_joint5" value="0" />
+    <joint name="robocol_joint5" value="1.19" />
+    <joint name="robocol_joint6" value="0" />
   </group_state>
   <!--END EFFECTOR: Purpose: Represent information about an end effector.-->

File: urdf/robocol_arm.urdf (robot description, URDF)
Before this commit: robot robocol, 7 links, 6 joints
Joints:
- joint robocol_joint1: limit lower=-3 upper=3 effort=87 velocity=2.3925 -> lower=-2.09 upper=2.09 effort=87 velocity=2.3925
- joint robocol_joint2: limit lower=-3 upper=3 effort=87 velocity=2.3925 -> lower=-1.75 upper=1.75 effort=87 velocity=2.3925
- joint robocol_joint3: limit lower=-3 upper=3 effort=87 velocity=2.3925 -> lower=-1.87 upper=2.76 effort=87 velocity=2.3925
- joint robocol_joint4: limit lower=-3 upper=3 effort=87 velocity=2.3925 -> lower=-2.97 upper=2.97 effort=87 velocity=2.3925
- joint robocol_joint5: limit lower=-3 upper=3 effort=12 velocity=2.8710 -> lower=-2.39 upper=1.75 effort=12 velocity=2.8710
- joint robocol_joint6: limit lower=-3 upper=3 effort=12 velocity=2.8710 -> lower=-2.97 upper=2.97 effort=12 velocity=2.8710

Commit message: Changes in package.xml

File: config/robocol_arm.xacro (robot description, xacro)
@@ -17,5 +17,5 @@
       <joint name="robocol_joint4" value="0" />
       <joint name="robocol_joint5" value="1.19" />
-      <!-- <joint name="robocol_joint6" value="0" /> -->
+      <joint name="robocol_joint6" value="0" />
     </group_state>
     <group_state name="ready" group="robocol_arm">
@@ -25,5 +25,5 @@
       <joint name="robocol_joint4" value="0" />
       <joint name="robocol_joint5" value="-0.78" />
-      <!-- <joint name="robocol_joint6" value="1.57" /> -->
+      <joint name="robocol_joint6" value="1.57" />
     </group_state>
     <group_state name="pick" group="robocol_arm">
@@ -33,5 +33,5 @@
       <joint name="robocol_joint4" value="0" />
       <joint name="robocol_joint5" value="0" />
-      <!-- <joint name="robocol_joint6" value="1.57" /> -->
+      <joint name="robocol_joint6" value="1.57" />
     </group_state>
     <group_state name="place_right" group="robocol_arm">
@@ -41,5 +41,5 @@
       <joint name="robocol_joint4" value="0" />
       <joint name="robocol_joint5" value="-0.95" />
-      <!-- <joint name="robocol_joint6" value="2.95" /> -->
+      <joint name="robocol_joint6" value="2.95" />
     </group_state>
     <group_state name="place_left" group="robocol_arm">
@@ -49,5 +49,5 @@
       <joint name="robocol_joint4" value="0" />
       <joint name="robocol_joint5" value="-0.95" />
-      <!-- <joint name="robocol_joint6" value="2.95" /> -->
+      <joint name="robocol_joint6" value="2.95" />
     </group_state>
     <group_state name="all_0" group="robocol_arm">
@@ -57,5 +57,5 @@
       <joint name="robocol_joint4" value="0" />
       <joint name="robocol_joint5" value="0" />
-      <!-- <joint name="robocol_joint6" value="0" /> -->
+      <joint name="robocol_joint6" value="0" />
     </group_state>
     <!--END EFFECTOR: Purpose: Represent information about an end effector.-->
@@ -68,4 +68,5 @@
     <disable_collisions link1="robocol_link3" link2="robocol_link4" reason="Adjacent" />
     <disable_collisions link1="robocol_link4" link2="robocol_link5" reason="Adjacent" />
+    <disable_collisions link1="robocol_link5" link2="robocol_link6" reason="Adjacent" />
     <!-- <disable_collisions link1="robocol_link2" link2="robocol_link3" reason="Adjacent" /> -->
     <disable_collisions link1="robocol_link0" link2="robocol_link2" reason="Never" />
